File: electronics/eeZeeTiny43U.brd (EAGLE design)
At the start: 36.3 x 20.3 mm, 15 parts, among them J2 avrisp

Commit message: don't recall
Routing:
- net !RESET: track 50.9 -> 50.0 mm
- net VCC: track 48.7 -> 48.1 mm
Changed lines of the file:
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@@
 <wire x1="18.288" y1="7.874" x2="20.154" y2="7.874" width="0.254" layer="1"/>
 <wire x1="20.154" y1="7.874" x2="20.828" y2="7.2" width="0.254" layer="1"/>
-<wire x1="18.288" y1="7.874" x2="18.288" y2="10.668" width="0.254" layer="1"/>
-<wire x1="18.288" y1="10.668" x2="17.526" y2="11.43" width="0.254" layer="1"/>
-<via x="17.526" y="11.43" extent="1-16" drill="0.3302"/>
-<wire x1="17.526" y1="11.43" x2="13.97" y2="11.43" width="0.254" layer="16"/>
-<via x="13.97" y="11.43" extent="1-16" drill="0.3302"/>
-<wire x1="13.97" y1="11.43" x2="4.484" y2="11.43" width="0.254" layer="1"/>
+<wire x1="18.288" y1="7.874" x2="18.288" y2="9.652" width="0.254" layer="1"/>
+<wire x1="18.288" y1="9.652" x2="17.526" y2="10.414" width="0.254" layer="1"/>
+<via x="17.526" y="10.414" extent="1-16" drill="0.3302"/>
+<wire x1="17.526" y1="10.414" x2="13.208" y2="10.414" width="0.254" layer="16"/>
+<via x="13.208" y="10.414" extent="1-16" drill="0.3302"/>
+<wire x1="13.208" y1="10.414" x2="8.636" y2="10.414" width="0.254" layer="1"/>
+<wire x1="8.636" y1="10.414" x2="7.62" y2="11.43" width="0.254" layer="1"/>
+<wire x1="7.62" y1="11.43" x2="4.484" y2="11.43" width="0.254" layer="1"/>
 <wire x1="4.484" y1="11.43" x2="4.318" y2="11.342" width="0.254" layer="1"/>
 <wire x1="32.258" y1="17.78" x2="30.988" y2="16.51" width="0.254" layer="1"/>
@@
 <wire x1="6.096" y1="15.494" x2="4.064" y2="15.494" width="0.254" layer="16"/>
 <wire x1="4.064" y1="15.494" x2="1.778" y2="17.78" width="0.254" layer="16"/>
-<wire x1="29.718" y1="12.7" x2="28.448" y2="12.7" width="0.254" layer="1"/>
-<wire x1="28.448" y1="12.7" x2="26.162" y2="10.414" width="0.254" layer="1"/>
-<via x="26.162" y="10.414" extent="1-16" drill="0.3302"/>
-<wire x1="26.162" y1="10.414" x2="11.176" y2="10.414" width="0.254" layer="16"/>
-<wire x1="11.176" y1="10.414" x2="6.096" y2="15.494" width="0.254" layer="16"/>
+<wire x1="29.718" y1="12.7" x2="27.432" y2="12.7" width="0.254" layer="1"/>
+<wire x1="27.432" y1="12.7" x2="26.162" y2="11.43" width="0.254" layer="1"/>
+<via x="26.162" y="11.43" extent="1-16" drill="0.3302"/>
+<wire x1="26.162" y1="11.43" x2="10.16" y2="11.43" width="0.254" layer="16"/>
+<wire x1="10.16" y1="11.43" x2="6.096" y2="15.494" width="0.254" layer="16"/>
 </signal>
 <signal name="PA6">
